File: uart.kicad_sch (KiCad schematic)
At the start: 11 parts, among them U7 MCP2200-I-SO, X1 12MHz

Commit message: asdasd
Parts:
- C10, C11: footprint (none) -> Capacitor_SMD:C_0201_0603Metric
- D2, D3: footprint LED_THT:LED_D3.0mm -> LED_SMD:LED_PLCC-2_3x2mm_AK
- X1: footprint (none) -> Oscillator:Oscillator_SMD_ECS_2520MV-xxx-xx-4Pin_2.5x2.0mm
Changed lines of the file:
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@@
 			)
 		)
-		(property "Footprint" ""
+		(property "Footprint" "Capacitor_SMD:C_0201_0603Metric"
 			(at 78.4352 71.12 0)
 			(effects
@@
 			)
 		)
-		(property "Footprint" ""
+		(property "Footprint" "Capacitor_SMD:C_0201_0603Metric"
 			(at 67.0052 71.12 0)
 			(effects
@@
 			)
 		)
-		(property "Footprint" "LED_THT:LED_D3.0mm"
+		(property "Footprint" "LED_SMD:LED_PLCC-2_3x2mm_AK"
 			(at 173.99 118.11 0)
 			(effects
@@
 			)
 		)
-		(property "Footprint" "LED_THT:LED_D3.0mm"
+		(property "Footprint" "LED_SMD:LED_PLCC-2_3x2mm_AK"
 			(at 165.1 118.11 0)
 			(effects
@@
 			)
 		)
-		(property "Footprint" ""
+		(property "Footprint" "Oscillator:Oscillator_SMD_ECS_2520MV-xxx-xx-4Pin_2.5x2.0mm"
 			(at 59.69 134.62 0)
 			(effects

Commit message: dasda
Connections:
- net RST: now reaches R4.2, U7.4 (RST)
Changed lines of the file:
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@@
+		)
+	)
+	(label "RST"
+		(at 135.89 95.25 0)
+		(fields_autoplaced yes)
+		(effects
+			(font
+				(size 1.27 1.27)
+			)
+			(justify left bottom)
 		)
 	)

Commit message: sdfdsf
Parts:
- added C16, C17: C, Capacitor_SMD:C_0201_0603Metric, symbol Device:C
- R4, R5, R6: footprint Resistor_SMD:R_0201_0603Metric -> Resistor_SMD:R_0603_1608Metric
- X1: value 12MHz -> 12M; footprint Oscillator:Oscillator_SMD_ECS_2520MV-xxx-xx-4Pin_2.5x2.0mm -> custom:73-XT49M1200-S
Connections:
- net +3.3V: now also C16.1, C17.1
- net GND: now also C16.2, C17.2

Commit message: asdfsa
Parts:
- removed C10, C16, C17: C, Capacitor_SMD:C_0201_0603Metric, symbol Device:C
- C11, C3, C4: footprint Capacitor_SMD:C_0201_0603Metric -> Capacitor_SMD:C_0603_1608Metric
Connections:
- net OSC1: now reaches C3.1, U7.2 (OSC1), X1.1
- net OSC2: now reaches C4.1, U7.3 (OSC2), X1.2
- net TX_LED: now reaches R5.1, U7.5 (GP7/TxLED)
- net RX_LED: now reaches R6.1, U7.6 (GP6/RxLED)
- net UART_CTS renamed UART2_CTS
- net UART_RTS renamed UART2_RTS
- net UART_RX renamed UART2_RX
- net UART_TX renamed UART2_TX
Other:
- moved on the sheet: C11, D2, D3, R5, R6

Commit message: asdfsa
Parts:
- added C10: 100n, Capacitor_SMD:C_0603_1608Metric, symbol Device:C
- added C12, C15, C16: 47p, Capacitor_SMD:C_0603_1608Metric, symbol Device:C
- added C6: 4u7, Capacitor_SMD:C_0603_1608Metric, symbol Device:C
- added D4, D5: LED, LED_SMD:LED_PLCC-2_3x2mm_AK, symbol Device:LED
- added FB1: FerriteBead, Capacitor_SMD:C_0603_1608Metric, symbol Device:FerriteBead
- added R14, R15: 270, Resistor_SMD:R_0603_1608Metric, symbol Device:R
- added R16, R17: 27, Resistor_SMD:R_0603_1608Metric, symbol Device:R
- added U8: FT230XS, Package_SO:SSOP-16_3.9x4.9mm_P0.635mm, symbol Interface_USB:FT230XS
Connections:
- net UART2_TX is gone; now on net UART2_RX: U7.10 (TX)
- net +3.3V: now also FB1.1
- net GND: now also C10.2, C12.2, C15.2, C16.2, C6.2, D4.1 (K), D5.1 (K), U8.12 (VCC), U8.13 (GND), U8.5 (GND)
- net RX_LED: now also R15.1, U8.14 (CBUS1)
- net TX_LED: now also R14.1, U8.7 (CBUS2)
- net UART2_CTS: now also U8.6 (~{CTS})
- net UART2_RTS: now also U8.2 (~{RTS})
- net UART2_RX: now also U8.1 (TXD), U8.4 (RXD)
- net USB_D+: now also C12.1, R16.1
- net USB_D-: now also C15.1, R17.2
- new net: R17.1, U8.8 (USBDP)
- new net: D5.2 (A), R15.2
- new net: C16.1, U8.10 (3V3OUT), U8.11 (~{RESET}), U8.3 (VCCIO)
- new net: D4.2 (A), R14.2
- new net: R16.2, U8.9 (USBDM)
- new net: C10.1, C6.1, FB1.2

Commit message: asdfsa
Parts:
- removed C11, C3, C4: C, Capacitor_SMD:C_0603_1608Metric, symbol Device:C
- removed D2, D3: LED, LED_SMD:LED_PLCC-2_3x2mm_AK, symbol Device:LED
- removed R4: 4k7, Resistor_SMD:R_0603_1608Metric, symbol Device:R
- removed R5, R6: R, Resistor_SMD:R_0603_1608Metric, symbol Device:R
- removed U7: MCP2200-I-SO, Package_SO:SOIC-20W_7.5x12.8mm_P1.27mm, symbol Interface_USB:MCP2200-I-SO
- removed X1: 12M, custom:73-XT49M1200-S, symbol Device:Crystal
Connections:
- net UART2_CTS renamed ~{UART2_CTS}
- net UART2_RTS renamed ~{UART2_RTS}
- no-connect marks 6 -> 0
