File: power_supply.kicad_sch (KiCad schematic)
At the start: 0 parts

Commit message: added usbc power supply
Parts:
- added C1: 1u, symbol Device:C
- added C2: 10u, symbol Device:C
- added D1: LED, symbol Device:LED
- added R1, R2: 5k1, symbol Device:R
- added R3: 2k2, symbol Device:R
- added U4: ~, symbol custom:UJ20-C-H-C-MSMT-TR (USB C 16 Pin)
- added U6: ~, symbol custom:TPS7B8333QDCYRQ1 (3.3V_LDO_Regulator)
Connections:
- new net: D1.2 (A), R3.2
- new net: R2.1, U4.B5 (CC2)
- new net: R1.1, U4.A5 (CC1)
- new net +3.3V: C2.1, R3.1, U6.3 (OUT)
- new net +5V: C1.1, U4.A4 (VBUS), U4.A9 (VBUS), U4.B4 (VBUS), U4.B9 (VBUS), U6.1 (IN)
- new net GND: C1.2, C2.2, D1.1 (K), R1.2, R2.2, U4.0 (SHELL), U4.A1 (GND), U4.A12 (GND), U4.B1 (GND), U4.B12 (GND), U6.2 (GND), U6.4 (GND)
- new net USB_D+: U4.A6 (DP1), U4.B6 (DP2)
- new net USB_D-: U4.A7 (DN1), U4.B7 (DN2)

Commit message: sdfdsf
Connections:
- net +5V: no longer U4.A4 (VBUS), U4.A9 (VBUS), U4.B4 (VBUS), U4.B9 (VBUS)
- new net +5V_USB: U4.A4 (VBUS), U4.A9 (VBUS), U4.B4 (VBUS), U4.B9 (VBUS)
Changed lines of the file:
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@@
+	)
+	(junction
+		(at 95.25 54.61)
+		(diameter 0)
+		(color 0 0 0 0)
 	)
 	(junction
@@
 	)
 	(junction
-		(at 95.25 54.61)
-		(diameter 0)
-		(color 0 0 0 0)
-	)
-	(junction
 		(at 167.64 64.77)
 		(diameter 0)
@@
 	(wire
 		(pts
+			(xy 95.25 49.53) (xy 95.25 54.61)
+		)
+		(stroke
+			(width 0)
+			(type default)
+		)
+	)
+	(wire
+		(pts
 			(xy 69.85 67.31) (xy 95.25 67.31)
 		)
@@
 		(pts
 			(xy 95.25 97.79) (xy 95.25 100.33)
-		)
-		(stroke
-			(width 0)
-			(type default)
-		)
-	)
-	(wire
-		(pts
-			(xy 95.25 49.53) (xy 95.25 54.61)
 		)
 		(stroke
@@
 	)
 	(symbol
-		(lib_id "power:+5V")
+		(lib_name "+5V_USB_1")
+		(lib_id "custom:+5V_USB")
 		(at 95.25 49.53 0)
 		(unit 1)
 		(exclude_from_sim no)
-		(in_bom yes)
-		(on_board yes)
+		(in_bom no)
+		(on_board no)
 		(dnp no)
 		(fields_autoplaced yes)
-		(property "Reference" "#PWR09"
-			(at 95.25 53.34 0)
-			(effects
-				(font
-					(size 1.27 1.27)
-				)
-				(hide yes)
-			)
-		)
-		(property "Value" "+5V"
+		(property "Reference" "#PWR021"
+			(at 95.25 49.53 0)
+			(effects
+				(font
+					(size 1.27 1.27)
+				)
+				(hide yes)
+			)
+		)
+		(property "Value" "+5V_USB"
 			(at 95.25 44.45 0)
 			(effects
@@
 			)
 		)
-		(property "Description" "Power symbol creates a global label with name \"+5V\""
+		(property "Description" ""
 			(at 95.25 49.53 0)
 			(effects
@@
 			(project ""
 				(path "/342e1e7c-839e-4cd3-a9c3-2caee679f2e5/13c5de07-3255-4d28-9ff7-29d107a6e2e5"
-					(reference "#PWR09")
+					(reference "#PWR021")
 					(unit 1)
 				)
@@
 					(unit 1)
 				)
+			)
+		)
+	)
+	(symbol
+		(lib_id "custom:+5V_USB")
+		(at 95.25 49.53 0)
+		(unit 1)
+		(exclude_from_sim no)
+		(in_bom no)
+		(on_board no)
+		(dnp no)
+		(fields_autoplaced yes)
+		(property "Reference" "#PWR09"
+			(at 95.25 44.45 0)
+			(effects
+				(font
+					(size 1.27 1.27)
+				)
+				(hide yes)
+			)
+		)
+		(property "Value" "+5V_USB"
+			(at 95.25 46.99 0)
+			(effects
+				(font
+					(size 1.27 1.27)
+				)
+				(hide yes)
+			)
+		)
+		(property "Footprint" ""
+			(at 95.25 49.53 0)
+			(effects
+				(font
+					(size 1.27 1.27)
+				)
+				(hide yes)
+			)
+		)
+		(property "Datasheet" ""
+			(at 95.25 49.53 0)
+			(effects
+				(font
+					(size 1.27 1.27)
+				)
+				(hide yes)
+			)
+		)
+		(property "Description" ""
+			(at 95.25 49.53 0)
+			(effects
+				(font
+					(size 1.27 1.27)
+				)
+				(hide yes)
+			)
+		)
+		(pin "1"
+		)
+		(instances
+			(project ""
+				(path "/342e1e7c-839e-4cd3-a9c3-2caee679f2e5/13c5de07-3255-4d28-9ff7-29d107a6e2e5"
+					(reference "#PWR09")
+					(unit 1)
+				)

Commit message: fsdf
Connections:
- net +5V: no longer names the net of C1.1, U6.1 (IN)

Commit message: dasda
Parts:
- C1, C2: footprint (none) -> Capacitor_SMD:C_0201_0603Metric
- D1: footprint (none) -> LED_THT:LED_D3.0mm
- R1, R2, R3: footprint (none) -> Resistor_SMD:R_0201_0603Metric
- U4: footprint (none) -> custom:UJ20-C-H-C-MSMT-TR
- U6: footprint (none) -> custom:TPS7B8333QDCYRQ1

Commit message: asdasd
Parts:
- D1: footprint LED_THT:LED_D3.0mm -> LED_SMD:LED_PLCC-2_3x2mm_AK
Connections:
- no-connect marks 0 -> 1
Changed lines of the file:
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@@
 		(color 0 0 0 0)
+	)
+	(no_connect
+		(at 25.4 80.01)
 	)
 	(wire
@@
 			)
 		)
-		(property "Footprint" "LED_THT:LED_D3.0mm"
+		(property "Footprint" "LED_SMD:LED_PLCC-2_3x2mm_AK"
 			(at 181.61 81.28 0)
 			(effects

Commit message: sdfdsf
Parts:
- R3: footprint Resistor_SMD:R_0201_0603Metric -> Resistor_SMD:R_0603_1608Metric
Changed lines of the file:
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@@
+		)
+	)
+	(label "USB_D+"
+		(at 72.39 74.93 0)
+		(fields_autoplaced yes)
+		(effects
+			(font
+				(size 1.27 1.27)
+			)
+			(justify left bottom)
+		)
+	)
+	(label "USB_D-"
+		(at 72.39 69.85 0)
+		(fields_autoplaced yes)
+		(effects
+			(font
+				(size 1.27 1.27)
+			)
+			(justify left bottom)
 		)
 	)
@@
 			)
 		)
-		(property "Footprint" "Resistor_SMD:R_0201_0603Metric"
+		(property "Footprint" "Resistor_SMD:R_0603_1608Metric"
 			(at 179.832 71.12 90)
 			(effects

Commit message: asdfsa
Parts:
- C1, C2: footprint Capacitor_SMD:C_0201_0603Metric -> Capacitor_SMD:C_0603_1608Metric
- R1, R2: footprint Resistor_SMD:R_0201_0603Metric -> Resistor_SMD:R_0603_1608Metric
Connections:
- net PWR_LED: now reaches D1.2 (A), R3.2
- net CC: now reaches R2.1, U4.B5 (CC2)
- net CC: now also R1.1, U4.A5 (CC1)
- no-connect marks 1 -> 3
Other:
- moved on the sheet: C1, C2, D1, R3

Commit message: asdfsa
Parts:
- R3: value 2k2 -> 270
Connections:
- net GND: no longer U4.0 (SHELL)
- no-connect marks 3 -> 4
Changed lines of the file:
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@@
-	)
-	(junction
-		(at 95.25 107.95)
-		(diameter 0)
-		(color 0 0 0 0)
 	)
 	(junction
@@
 		(at 60.96 90.17)
 	)
+	(no_connect
+		(at 60.96 107.95)
+	)
 	(wire
 		(pts
@@
 	(wire
 		(pts
-			(xy 60.96 107.95) (xy 95.25 107.95)
-		)
-		(stroke
-			(width 0)
-			(type default)
-		)
-	)
-	(wire
-		(pts
 			(xy 167.64 64.77) (xy 181.61 64.77)
 		)
@@
 	(wire
 		(pts
-			(xy 95.25 107.95) (xy 95.25 118.11)
+			(xy 95.25 105.41) (xy 95.25 118.11)
 		)
 		(stroke
@@
 		(pts
 			(xy 181.61 64.77) (xy 181.61 71.12)
-		)
-		(stroke
-			(width 0)
-			(type default)
-		)
-	)
-	(wire
-		(pts
-			(xy 95.25 105.41) (xy 95.25 107.95)
 		)
 		(stroke
@@
 			)
 		)
-		(property "Value" "2k2"
+		(property "Value" "270"
 			(at 184.15 76.1999 0)
 			(effects
