File: power_supply.kicad_sch (KiCad schematic)
At the start: 16 parts, among them U7 FT230XS

Commit message: fsdgds
Connections:
- net +3.3V: now also R18.1, R6.1
- net GND: no longer D2.1 (K), D3.1 (K)
- net RX_LED: now also D3.1 (K); no longer R18.1
- net TX_LED: now also D2.1 (K); no longer R6.1
Other:
- moved on the sheet: D2, D3, R18, R6

Commit message: adsad
Parts:
- removed C18: 4u7, Capacitor_SMD:C_0603_1608Metric, symbol Device:C
- added R14, R3: 120, Resistor_SMD:R_0603_1608Metric, symbol Device:R
- C11: value 47p -> 100n
- FB2: value FerriteBead -> 10u
Connections:
- net GND: no longer U7.12 (VCC)
- net UART2_RX: now also R3.1, R3.2
- net UART2_TX: now also R14.1, R14.2
- net at C17.1: now also FB2.2, U7.12 (VCC); no longer FB2.1
Other:
- moved on the sheet: C17, FB2
