File: power_supply.kicad_sch (KiCad schematic)
At the start: 17 parts, among them U7 FT230XS

Commit message: fsdf
Parts:
- added D1: LED, LED_SMD:LED_PLCC-2_3x2mm_AK, symbol Device:LED
- added R17: 270, Resistor_SMD:R_0603_1608Metric, symbol Device:R
Connections:
- net +3.3V: now also R17.1
- net GND: now also D1.1 (K)
- net CC renamed CC1
- net CC1: no longer R2.1, U4.B5 (CC2)
- new net: D1.2 (A), R17.2
- new net CC2: R2.1, U4.B5 (CC2)
Other:
- note added: "Power LED"

Commit message: fsdfsdf
Connections:
- net +3.3V: now also C11.1, U7.11 (~{RESET})
Changed lines of the file:
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@@
+	)
+	(junction
+		(at 177.8 90.17)
+		(diameter 0)
+		(color 0 0 0 0)
 	)
 	(junction
@@
 	)
 	(junction
+		(at 177.8 105.41)
+		(diameter 0)
+		(color 0 0 0 0)
+	)
+	(junction
 		(at 95.25 105.41)
 		(diameter 0)
@@
 		)
 		(stroke
+			(width 0)
+			(type default)
+		)
+	)
+	(wire
+		(pts
+			(xy 177.8 90.17) (xy 177.8 105.41)
+		)
+		(stroke

Commit message: fsdfsdf
Parts:
- removed U4: ~, custom:640-USB4215-03-A, symbol custom:UJ20-C-H-C-MSMT-TR (USB C 16 Pin)
- added J4: USB_C_Receptacle_USB2.0_16P, custom:640-USB4215-03-A, symbol Connector:USB_C_Receptacle_USB2.0_16P
Connections:
- net +5V_USB: now also J4.A4 (VBUS), J4.A9 (VBUS), J4.B4 (VBUS), J4.B9 (VBUS)
- net CC1: now also J4.A5 (CC1)
- net CC2: now also J4.B5 (CC2)
- net GND: now also J4.A1 (GND), J4.A12 (GND), J4.B1 (GND), J4.B12 (GND), J4.S1 (SHIELD)
- net RX_LED: now also D3.2 (A), R18.2
- net TX_LED: now also D2.2 (A), R6.2
- net USB_D+: now also J4.A6 (D+), J4.A7 (D-), J4.B6 (D+), J4.B7 (D-)
- net PWR_LED: now reaches D1.2 (A), R17.2
- no-connect marks 6 -> 4
Other:
- note removed: "Power LED"
- moved on the sheet: C11, C17, C3, C4, D1, D2, D3, FB2, R1, R14, R17, R18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

Commit message: asdsad
Parts:
- added C6: 100n, Capacitor_SMD:C_0603_1608Metric, symbol Device:C
- added U6: USBLC6-2SC6, Package_TO_SOT_SMD:SOT-23-6, symbol Power_Protection:USBLC6-2SC6
Connections:
- net +5V_USB: now also C6.1, U6.5 (VBUS)
- net GND: now also C6.2, U6.2 (GND)
- net USB_D+: now also U6.1 (I/O1), U6.3 (I/O2), U6.4 (I/O2), U6.6 (I/O1)
