File: mcu.kicad_sch (KiCad schematic)
At the start: 13 parts, among them SW1 SW_Nidec_CAS-120A1, SW2 SW_Push, U1 STM32G0B0KETx

Commit message: sdfdsf
Parts:
- added J1, J3: Conn_01x04_Pin, Connector_PinHeader_2.54mm:PinHeader_1x04_P2.54mm_Vertical, symbol Connector:Conn_01x04_Pin
- added J2: Conn_01x06_Pin, Connector_PinHeader_2.54mm:PinHeader_1x06_P2.54mm_Vertical, symbol Connector:Conn_01x06_Pin
- added R7: 10k, Resistor_SMD:R_0603_1608Metric, symbol Device:R
Connections:
- net +3.3V: now also J1.1 (Pin_1), J2.1 (Pin_1), J3.1 (Pin_1)
- net BOOT0: now also J1.2 (Pin_2), R7.2; no longer SW1.2 (B)
- net GND: now also J1.4 (Pin_4), J2.6 (Pin_6), J3.4 (Pin_4)
- net UART1_TX: now reaches U1.19 (PA9/NC)
- net UART1_TX: now also J2.5 (Pin_5)
- net UART1_RX: now reaches U1.21 (PA10/NC)
- net UART1_RX: now also J2.4 (Pin_4)
- net UART1_CTS: now reaches U1.22 (PA11/PA9)
- net UART1_CTS: now also J2.3 (Pin_3)
- net UART1_RTS: now reaches U1.23 (PA12/PA10)
- net UART1_RTS: now also J2.2 (Pin_2)
- net SWDIO: now reaches U1.24 (PA13)
- net SWDIO: now also J1.3 (Pin_3)
- net I2C1_SDA: now reaches U1.31 (PB7)
- net I2C1_SDA: now also J3.3 (Pin_3)
- net I2C1_SCL: now reaches U1.32 (PB8)
- net I2C1_SCL: now also J3.2 (Pin_2)
- new net: R7.1, SW1.2 (B)
- no-connect marks 30 -> 23
Other:
- note added: "I2C1"
- note added: "SERIAL WIRE DEBUG"
- note added: "UART1"

Commit message: asdfsa
Parts:
- removed C15: 100u, Capacitor_SMD:C_0201_0603Metric, symbol Device:C
- added R10: 10k, Resistor_SMD:R_0603_1608Metric, symbol Device:R
- C13, C14, C8, C9: footprint Capacitor_SMD:C_0201_0603Metric -> Capacitor_SMD:C_0603_1608Metric
Connections:
- net +3.3V: now also R10.2
- net BOOT0: now also R7.1, SW1.2 (B)
- net FLASH_CS: now also R10.1
- net FLASH_NAND_CS renamed FLASH_NOR_CS

Commit message: asdfsa
Parts:
- added R11: 22, Resistor_SMD:R_0603_1608Metric, symbol Device:R
- added R12, R13: 5k1, Resistor_SMD:R_0603_1608Metric, symbol Device:R
- R10: value 10k -> 56k
Connections:
- net +3.3V: now also R12.2, R13.2
- net I2C1_SCL: now also R12.1
- net I2C1_SDA: now also R13.1
- net SPI1_SCK: now also R11.1, R11.2
Other:
- moved on the sheet: C8, C9, H1, H2, H3, H4, R10, U1

Commit message: asdfsa
Connections:
- net +3.3V: no longer U1.4 (VDD)
- net GND: now also U1.4 (VDD)
- net UART1_CTS renamed ~{UART1_CTS}
- net UART1_RTS renamed ~{UART1_RTS}
- net UART2_CTS renamed ~{UART2_CTS}
- net UART2_RTS renamed ~{UART2_RTS}
Other:
- moved on the sheet: C8, C9, J1, J2, J3, R10, R11, R12, R13, U1

Commit message: adsad
Parts:
- added R15, R16: 120, Resistor_SMD:R_0603_1608Metric, symbol Device:R
- C13, C14, C9: value C -> 100n
- R12, R13: value 5k1 -> 1k8
Connections:
- net UART1_RX: now also R16.2; no longer J2.4 (Pin_4)
- net UART1_TX: now also R15.1; no longer J2.5 (Pin_5)
- new net: J2.4 (Pin_4), R16.1
- new net: J2.5 (Pin_5), R15.2
Other:
- moved on the sheet: C8, C9, J1, J2, J3, R10, R11, R12, R13, U1
