File: mcu.kicad_sch (KiCad schematic)
At the start: 22 parts, among them J1 Conn_01x04_Pin, J2 Conn_01x06_Pin, J3 Conn_01x04_Pin, SW1 SW_Nidec_CAS-120A1, SW2 SW_Push, U1 STM32G0B0KETx

Commit message: fsdf
Parts:
- added C1: 100n, Capacitor_SMD:C_0603_1608Metric, symbol Device:C
- added D4: LED, LED_SMD:LED_PLCC-2_3x2mm_AK, symbol Device:LED
- added R19: 270, Resistor_SMD:R_0603_1608Metric, symbol Device:R
- added R20, R21: 10k, Resistor_SMD:R_0603_1608Metric, symbol Device:R
- added SW3: SW_Push, Button_Switch_SMD:SW_Push_SPST_NO_Alps_SKRK, symbol Switch:SW_Push
Connections:
- net +3.3V: now also R20.2, SW3.1
- net GND: now also C1.2, D4.1 (K)
- net USER_BTN: now reaches U1.1 (PB9)
- net USER_BTN: now also R21.1
- net USER_LED: now reaches U1.16 (PB1)
- net USER_LED: now also R19.1
- new net: D4.2 (A), R19.2
- new net: C1.1, R20.1, R21.2, SW3.2
- no-connect marks 23 -> 21
Other:
- note added: "User LED"
- moved on the sheet: C8, C9, J1, J2, J3, R10, R11, R12, R13, R15, R16, U1

Commit message: fsdfsdf
Parts:
- C8: value 100u -> 10u
Other:
- note removed: "SPI Series resistors next time"
- moved on the sheet: D4, R19
Changed lines of the file:
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@@
 	(wire
 		(pts
-			(xy 119.38 54.61) (xy 119.38 57.15)
+			(xy 193.04 50.8) (xy 193.04 53.34)
 		)
 		(stroke
@@
 	(wire
 		(pts
-			(xy 113.03 40.64) (xy 119.38 40.64)
+			(xy 186.69 36.83) (xy 193.04 36.83)
 		)
 		(stroke
@@
 	(wire
 		(pts
-			(xy 119.38 40.64) (xy 119.38 46.99)
+			(xy 193.04 36.83) (xy 193.04 43.18)
 		)
 		(stroke
@@
 	(wire
 		(pts
-			(xy 119.38 64.77) (xy 119.38 68.58)
+			(xy 193.04 60.96) (xy 193.04 64.77)
 		)
 		(stroke
@@
 	(text "User LED\n"
 		(exclude_from_sim no)
-		(at 111.76 60.96 0)
-		(effects
-			(font
-				(size 1.27 1.27)
-			)
-		)
-	)
-	(text "SPI Series resistors next time"
-		(exclude_from_sim no)
-		(at 193.294 75.438 0)
+		(at 185.42 57.15 0)
 		(effects
 			(font
@@
 	(global_label "USER_LED"
 		(shape input)
-		(at 113.03 40.64 180)
+		(at 186.69 36.83 180)
 		(fields_autoplaced yes)
 		(effects
@@
 		)
 		(property "Intersheetrefs" "${INTERSHEET_REFS}"
-			(at 100.6711 40.64 0)
+			(at 174.3311 36.83 0)
 			(effects
 				(font
@@
 	(symbol
 		(lib_id "Device:LED")
-		(at 119.38 60.96 90)
+		(at 193.04 57.15 90)
 		(unit 1)
 		(exclude_from_sim no)
@@
 		(fields_autoplaced yes)
 		(property "Reference" "D4"
-			(at 123.19 61.2774 90)
+			(at 196.85 57.4674 90)
 			(effects
 				(font
@@
 		)
 		(property "Value" "LED"
-			(at 123.19 63.8174 90)
+			(at 196.85 60.0074 90)
 			(effects
 				(font
@@
 		)
 		(property "Footprint" "LED_SMD:LED_PLCC-2_3x2mm_AK"
-			(at 147.32 36.83 0)
+			(at 220.98 33.02 0)
 			(effects
 				(font
@@
 		)
 		(property "Datasheet" "~"
-			(at 119.38 60.96 0)
+			(at 193.04 57.15 0)
 			(effects
 				(font
@@
 		)
 		(property "Description" "Light emitting diode"
-			(at 119.38 60.96 0)
+			(at 193.04 57.15 0)
 			(effects
 				(font
@@
 			)
 		)
-		(property "Value" "100u"
+		(property "Value" "10u"
 			(at 148.59 62.2299 0)
 			(effects
@@
 	(symbol
 		(lib_id "Device:R")
-		(at 119.38 50.8 0)
+		(at 193.04 46.99 0)
 		(unit 1)
 		(exclude_from_sim no)
@@
 		(fields_autoplaced yes)
 		(property "Reference" "R19"
-			(at 121.92 49.5299 0)
+			(at 195.58 45.7199 0)
 			(effects
 				(font
@@
 		)
 		(property "Value" "270"
-			(at 121.92 52.0699 0)
+			(at 195.58 48.2599 0)
 			(effects
 				(font
@@
 		)
 		(property "Footprint" "Resistor_SMD:R_0603_1608Metric"
-			(at 145.542 26.67 90)
+			(at 219.202 22.86 90)
 			(effects
 				(font
@@
 		)
 		(property "Datasheet" "~"
-			(at 119.38 50.8 0)
+			(at 193.04 46.99 0)
 			(effects
 				(font
@@
 		)
 		(property "Description" "Resistor"
-			(at 119.38 50.8 0)
+			(at 193.04 46.99 0)
 			(effects
 				(font
@@
 	(symbol
 		(lib_id "power:GND")
-		(at 119.38 68.58 0)
+		(at 193.04 64.77 0)
 		(unit 1)
 		(exclude_from_sim no)
@@
 		(fields_autoplaced yes)
 		(property "Reference" "#PWR015"
-			(at 119.38 74.93 0)
+			(at 193.04 71.12 0)
 			(effects
 				(font
@@
 		)
 		(property "Value" "GND"
-			(at 119.38 73.66 0)
+			(at 193.04 69.85 0)
 			(effects
 				(font
@@
 		)
 		(property "Footprint" ""
-			(at 119.38 68.58 0)
+			(at 193.04 64.77 0)
 			(effects
 				(font
@@
 		)
 		(property "Datasheet" ""
-			(at 119.38 68.58 0)
+			(at 193.04 64.77 0)
 			(effects
 				(font
@@
 		)
 		(property "Description" "Power symbol creates a global label with name \"GND\" , ground"
-			(at 119.38 68.58 0)
+			(at 193.04 64.77 0)
 			(effects
 				(font

Commit message: sadsad
Connections:
- net +3.3V: no longer SW3.1
- net GND: now also SW3.1
- net USER_BTN: now also U5.6 (O_{2}); no longer R21.1
- net at R20.1, R21.2, SW3.2: no longer C1.1
- net ~{USER_BTN}: now reaches U5.5 (I_{2})
- net ~{USER_BTN}: now also C1.1, R21.1
- no-connect marks 21 -> 19
Other:
- note added: "R21 auch 1k?"
- moved on the sheet: C1, C14, R20, R21, SW3

Commit message: fsdfsdf
Parts:
- removed J1, J3: Conn_01x04_Pin, Connector_PinHeader_2.54mm:PinHeader_1x04_P2.54mm_Vertical, symbol Connector:Conn_01x04_Pin
- removed J2: Conn_01x06_Pin, Connector_PinHeader_2.54mm:PinHeader_1x06_P2.54mm_Vertical, symbol Connector:Conn_01x06_Pin
- removed U5: ~, custom:74AC14SCX, symbol custom:74AC14SCX
- added J5, J7: Conn_01x12_Pin, Connector_PinHeader_2.54mm:PinHeader_1x12_P2.54mm_Vertical, symbol Connector:Conn_01x12_Pin
- added R22, R23: 1k8, Resistor_SMD:R_0603_1608Metric, symbol Device:R
- added U4: ~, custom:74HC3G14-Q100, symbol custom:74HC3G14DC-Q100H
- R10: value 56k -> 10k
- R12: value 1k8 -> 56k
- R13: value 1k8 -> 10k
Connections:
- net +3.3V: now also U1.4 (VDD), J5.1 (Pin_1), J7.1 (Pin_1), R22.2, R23.2, U4.8 (VCC); no longer R13.2
- net BOOT0: now also J5.6 (Pin_6)
- net FLASH_CS: now also R12.1, U4.1 (1A); no longer R10.1
- net FLASH_NOR_CS: now also U4.7 (1Y)
- net GND: now also J5.11 (Pin_11), J5.12 (Pin_12), J7.12 (Pin_12), U4.4 (GND); no longer U1.4 (VDD)
- net I2C1_SCL: now also J7.3 (Pin_3), R23.1; no longer R12.1
- net I2C1_SDA: now also J7.2 (Pin_2), R22.1; no longer R13.1
- net NRST: now also U4.5 (2Y); no longer C13.2, SW2.2
- net SWDIO: now also J5.7 (Pin_7)
- net USER_BTN: now also U4.2 (3Y)
- net ~{UART1_CTS}: now also J5.3 (Pin_3)
- net ~{UART1_RTS}: now also J5.2 (Pin_2)
- net ~{USER_BTN}: now also U4.6 (3A)
- net at R16.1: now also J5.4 (Pin_4)
- net at R15.2: now also J5.5 (Pin_5)
- net PB0: now reaches U1.15 (PB0)
- net PB0: now also J7.7 (Pin_7)
- net PB2: now reaches U1.17 (PB2)
- net PB2: now also J7.8 (Pin_8)
- net PA8: now reaches U1.18 (PA8)
- net PA8: now also J5.8 (Pin_8)
- net PC14: now reaches U1.2 (PC14)
- net PC14: now also J7.5 (Pin_5)
- net PC6: now reaches U1.20 (PC6)
- net PC6: now also J7.4 (Pin_4)
- net PA15: now reaches U1.26 (PA15)
- net PA15: now also J5.9 (Pin_9)
- net PB3: now reaches U1.27 (PB3)
- net PB3: now also J7.9 (Pin_9)
- net PB4: now reaches U1.28 (PB4)
- net PB4: now also J7.10 (Pin_10)
- net PB5: now reaches U1.29 (PB5)
- net PB5: now also J7.11 (Pin_11)
- net PC15: now reaches U1.3 (PC15)
- net PC15: now also J7.6 (Pin_6)
- net PB6: now reaches U1.30 (PB6)
- net PB6: now also J5.10 (Pin_10)
- new net: R10.1, R13.2, SW2.2
- new net RST: C13.2, R13.1, U4.3 (2A)
- no-connect marks 19 -> 0
Other:
- note removed: "I2C1"
- note removed: "SERIAL WIRE DEBUG"
- note removed: "UART1"
- moved on the sheet: C13, C8, C9, D4, H1, H2, H3, H4, R11, R15, R16, R19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

Commit message: asdsad
Parts:
- removed R10: 10k, Resistor_SMD:R_0603_1608Metric, symbol Device:R
- removed R15, R16: 120, Resistor_SMD:R_0603_1608Metric, symbol Device:R
- removed R22, R23: 1k8, Resistor_SMD:R_0603_1608Metric, symbol Device:R
- removed U4: ~, custom:74HC3G14-Q100, symbol custom:74HC3G14DC-Q100H
- added C2: 100n, Capacitor_SMD:C_0603_1608Metric, symbol Device:C
- added D5: D, Diode_SMD:D_0603_1608Metric, symbol Device:D
- added U4, U5: SN74LVC1G14DBV, Package_TO_SOT_SMD:SOT-23-5, symbol 74xGxx:SN74LVC1G14DBV
Connections:
- net RST is gone; now on net NRST: C13.2, R13.1
- net UART1_TX is gone; now on net PA9: U1.19 (PA9/NC)
- net +3.3V: now also C2.2, U4.5 (VCC), U5.5 (VCC)
- net BOOT0: now also J5.11 (Pin_11); no longer J5.6 (Pin_6)
- net FLASH_CS: now also U4.2
- net FLASH_NOR_CS: now also U4.4
- net GND: now also C2.1, U4.3 (GND), U5.3 (GND); no longer J5.11 (Pin_11)
- net PA15: now also J7.10 (Pin_10); no longer J5.9 (Pin_9)
- net PA8: now also J5.4 (Pin_4); no longer J5.8 (Pin_8)
- net PB0: now also J5.2 (Pin_2); no longer J7.7 (Pin_7)
- net PB2: now also J5.3 (Pin_3); no longer J7.8 (Pin_8)
- net PB4: now also J7.8 (Pin_8); no longer J7.10 (Pin_10)
- net PB5: now also J7.7 (Pin_7); no longer J7.11 (Pin_11)
- net PB6: now also J7.6 (Pin_6); no longer J5.10 (Pin_10)
- net PC14: now also J7.3 (Pin_3); no longer J7.5 (Pin_5)
- net PC15: now also J7.2 (Pin_2); no longer J7.6 (Pin_6)
- net PC6: now also J5.6 (Pin_6); no longer J7.4 (Pin_4)
- net SWDIO: now also J5.10 (Pin_10); no longer J5.7 (Pin_7)
- net USER_BTN: now also U5.4
- net NRST_PIN: now reaches R13.2, SW2.2
- net NRST_PIN: now also J7.11 (Pin_11)
- net at R20.1, R21.2, SW3.2: now also D5.2 (A)
- net PA9: now reaches J5.5 (Pin_5)
- net I2C1_SCL renamed PB8
- net PB8: now also J7.4 (Pin_4); no longer J7.3 (Pin_3)
- net I2C1_SDA renamed PB7
- net PB7: now also J7.5 (Pin_5); no longer J7.2 (Pin_2)
- net UART1_RX renamed PA10
- net PA10: now also J5.7 (Pin_7)
- net ~{UART1_CTS} renamed PA11
- net PA11: now also J5.8 (Pin_8); no longer J5.3 (Pin_3)
- net ~{UART1_RTS} renamed PA12
- net PA12: now also J5.9 (Pin_9); no longer J5.2 (Pin_2)
- net ~{USER_BTN}: no longer names the net of C1.1, R21.1
- net ~{USER_BTN}: now also D5.1 (K), U5.2
Other:
- note removed: "R21 auch 1k?"
- moved on the sheet: C13, R12, R13, R20, SW2
