File: stm32G0_mcu.kicad_pcb (KiCad board)
At the start: 4 copper layers, 75 x 40 mm, 38 parts, among them SW1 SW_Nidec_CAS-120A1, SW2 SW_Push, U1 STM32G0B0KETx, U7 MCP2200-I-SO, X1 12MHz

Commit message: sdfdsf
Parts:
- added C16: C, Capacitor_SMD:C_0201_0603Metric, F.Cu at (102.8, 95.5)
- added C17: C, Capacitor_SMD:C_0201_0603Metric, F.Cu at (102.8, 96.9)
- added J1: Conn_01x04_Pin, Connector_PinHeader_2.54mm:PinHeader_1x04_P2.54mm_Vertical, F.Cu at (122.5, 71.0)
- added J2: Conn_01x06_Pin, Connector_PinHeader_2.54mm:PinHeader_1x06_P2.54mm_Vertical, F.Cu at (135.7, 71.0)
- added J3: Conn_01x04_Pin, Connector_PinHeader_2.54mm:PinHeader_1x04_P2.54mm_Vertical, F.Cu at (109.2, 71.0)
- added R7: 10k, Resistor_SMD:R_0603_1608Metric, F.Cu at (119.2, 80.6)
- R3, R4, R5, R6: footprint Resistor_SMD:R_0201_0603Metric -> Resistor_SMD:R_0603_1608Metric
- X1: value 12MHz -> 12M; footprint Oscillator:Oscillator_SMD_ECS_2520MV-xxx-xx-4Pin_2.5x2.0mm -> custom:73-XT49M1200-S
- moved SW1 31.8 mm to (96.2, 71.9)
- moved R4 12.4 mm to (106.9, 96.7), turned to 90 degrees
- moved C3 10.0 mm to (99.3, 105.8)
- moved C10 8.50 mm to (108.6, 81.9), turned to 90 degrees
- moved D1 8.34 mm to (105.3, 77.4)
- moved R3 8.33 mm to (100.9, 77.3)
- moved C11 8.24 mm to (106.9, 81.9), turned to 90 degrees
- moved R5 5.25 mm to (116.9, 99.4)
- moved R6 5.14 mm to (121.6, 99.5)
- moved C4 4.78 mm to (112.1, 105.9)
- moved U7 2.95 mm to (108.8, 88.9), turned to 90 degrees
- moved X1 2.90 mm to (105.8, 102.4), turned to 0 degrees
- moved C8 2.22 mm to (121.8, 90.6), turned to -90 degrees
- moved C12 2.19 mm to (139.4, 92.4), turned to 180 degrees
- moved C6 2.18 mm to (139.5, 77.8), turned to 180 degrees
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Connections:
- C1 pad 1: +5V_USB -> Net-(U6-IN)
- C3 pad 1: +3.3V -> OSC
- C4 pad 1: +3.3V -> OSC
- D1 pad 2: +3.3V -> Net-(D1-A)
- D2 pad 2: +3.3V -> TxLED
- D3 pad 2: +3.3V -> RxLED
- R3 pad 2: +3.3V -> Net-(D1-A)
- R5 pad 1: +3.3V -> TxLED
- R5 pad 2: +3.3V -> TxLED
- R6 pad 1: +3.3V -> RxLED
- R6 pad 2: +3.3V -> RxLED
- SW1 pad 2: BOOT0 -> Net-(SW1-B)
- U1 pad 10: UART2_RX -> UART_RX
- U1 pad 19: unconnected-(U1-PA9/NC-Pad19) -> UART1_TX
- U1 pad 21: unconnected-(U1-PA10/NC-Pad21) -> UART1_RX
- U1 pad 22: unconnected-(U1-PA11/PA9-Pad22) -> UART1_CTS
- U1 pad 23: unconnected-(U1-PA12/PA10-Pad23) -> UART1_RTS
- U1 pad 24: unconnected-(U1-PA13-Pad24) -> SWDIO
- U1 pad 31: unconnected-(U1-PB7-Pad31) -> I2C1_SDA
- U1 pad 32: unconnected-(U1-PB8-Pad32) -> I2C1_SCL
- U2 pad 15: SPI1_MOSI -> /FLASH/SPI10
- U2 pad 8: SPI1_MISO -> /FLASH/SPI11
- U3 pad 15: SPI1_MOSI -> /FLASH/SPI10
- U3 pad 8: SPI1_MISO -> /FLASH/SPI11
- U4 pad A5: GND -> Net-(U4-CC1)
- U4 pad A8: GND -> unconnected-(U4-SBU1-PadA8)
- U4 pad B5: GND -> Net-(U4-CC2)
- U4 pad B8: GND -> unconnected-(U4-SBU2-PadB8)
- U6 pad 1: +5V_USB -> Net-(U6-IN)
- U7 pad 2: +3.3V -> OSC
- U7 pad 3: +3.3V -> OSC
- U7 pad 5: +3.3V -> TxLED
- U7 pad 6: +3.3V -> RxLED
- X1 pad 1: +3.3V -> OSC
- X1 pad 2: +3.3V -> OSC
Routing:
- net +3.3V: track 128.6 -> 44.0 mm, vias 10 -> 11
- net OSC: track 0.00 -> 36.0 mm
- net UART_RX: track 0.00 -> 29.9 mm, vias 0 -> 2
- net UART1_TX: track 0.00 -> 29.8 mm
- net Net-(SW1-B): track 0.00 -> 26.2 mm, vias 0 -> 2
- net UART1_RX: track 0.00 -> 26.2 mm
- net I2C1_SCL: track 0.00 -> 25.5 mm
- net UART_CTS: track 0.00 -> 24.6 mm
- net I2C1_SDA: track 0.00 -> 23.8 mm
- net UART1_CTS: track 0.00 -> 23.0 mm
- net UART_RTS: track 0.00 -> 21.7 mm
- net UART1_RTS: track 0.00 -> 20.1 mm
- net SWDIO: track 0.00 -> 19.9 mm
- net RxLED: track 0.00 -> 18.1 mm
- net BOOT0: track 11.2 -> 27.0 mm, vias 0 -> 2
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Other:
- board text added: "PWR"
- board text added: "SWD"
- board text added: "UART2"
- board text removed: "POWER"

Commit message: asdfsa
Parts:
- removed C10, C12, C16, C17, C6: C, Capacitor_SMD:C_0201_0603Metric
- removed C15: 100u, Capacitor_SMD:C_0201_0603Metric
- added R10: 10k, Resistor_SMD:R_0603_1608Metric, F.Cu at (137.1, 110.5)
- added R8: 10k, Resistor_SMD:R_0603_1608Metric, F.Cu at (148.3, 107.6)
- added R9: 10k, Resistor_SMD:R_0603_1608Metric, F.Cu at (148.5, 92.9)
- C1, C11, C13, C14, C2, C3, C4, C8, C9: footprint Capacitor_SMD:C_0201_0603Metric -> Capacitor_SMD:C_0603_1608Metric
- C5, C7: value C -> 220n; footprint Capacitor_SMD:C_0201_0603Metric -> Capacitor_SMD:C_0603_1608Metric
- R1, R2: footprint Resistor_SMD:R_0201_0603Metric -> Resistor_SMD:R_0603_1608Metric
- moved C7 31.2 mm to (163.3, 114.4), turned to 90 degrees
- moved C5 31.2 mm to (163.3, 99.8), turned to 90 degrees
- moved C14 26.0 mm to (145.1, 117.8), turned to 90 degrees
- moved H3 22.4 mm to (165.0, 125.0)
- moved R6 21.7 mm to (129.9, 119.5)
- moved D2 21.7 mm to (125.3, 124.0)
- moved D3 21.7 mm to (129.9, 124.0)
- moved R5 21.7 mm to (125.2, 119.4)
- moved H4 21.5 mm to (95.0, 125.0)
- moved U5 21.3 mm to (140.6, 122.4), turned to -90 degrees
- moved C3 20.0 mm to (106.5, 124.5)
- moved C4 20.0 mm to (119.2, 124.6)
- moved R3 19.2 mm to (105.0, 96.1), turned to 90 degrees
- moved U4 19.1 mm to (93.3, 105.0)
- moved X1 18.7 mm to (112.9, 119.7)
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Connections:
- net Net-(D1-A) renamed /POWER_SUPPLY/PWR_LED
- net UART_RX renamed UART2_RX
- C1 pad 1: Net-(U6-IN) -> +5V_USB
- C3 pad 1: OSC -> /UART/OSC1
- C4 pad 1: OSC -> /UART/OSC2
- D2 pad 2: TxLED -> Net-(D2-A)
- D3 pad 2: RxLED -> Net-(D3-A)
- R1 pad 1: Net-(U4-CC1) -> /POWER_SUPPLY/CC
- R2 pad 1: Net-(U4-CC2) -> /POWER_SUPPLY/CC
- R5 pad 1: TxLED -> /UART/TX_LED
- R5 pad 2: TxLED -> Net-(D2-A)
- R6 pad 1: RxLED -> /UART/RX_LED
- R6 pad 2: RxLED -> Net-(D3-A)
- R7 pad 1: Net-(SW1-B) -> BOOT0
- SW1 pad 2: Net-(SW1-B) -> BOOT0
- U2 pad 1: unconnected-(U2-HOLD(IO_{3})-Pad1) -> Net-(U2-HOLD(IO_{3}))
- U2 pad 15: /FLASH/SPI10 -> SPI1_MOSI
- U2 pad 7: FLASH_NAND_CS -> FLASH_CS
- U2 pad 8: /FLASH/SPI11 -> SPI1_MISO
- U2 pad 9: unconnected-(U2-WP(IO_{2})-Pad9) -> Net-(U2-HOLD(IO_{3}))
- U3 pad 1: unconnected-(U3-HOLD(IO_{3})-Pad1) -> Net-(U3-HOLD(IO_{3}))
- U3 pad 15: /FLASH/SPI10 -> SPI1_MOSI
- U3 pad 7: FLASH_CS -> FLASH_NOR_CS
- U3 pad 8: /FLASH/SPI11 -> SPI1_MISO
- U3 pad 9: unconnected-(U3-WP(IO_{2})-Pad9) -> Net-(U3-HOLD(IO_{3}))
- U4 pad A5: Net-(U4-CC1) -> /POWER_SUPPLY/CC
- U4 pad B5: Net-(U4-CC2) -> /POWER_SUPPLY/CC
- U5 pad 2: FLASH_NAND_CS -> FLASH_NOR_CS
- U6 pad 1: Net-(U6-IN) -> +5V_USB
- U7 pad 10: UART_TX -> UART2_TX
- U7 pad 11: UART_RTS -> UART2_RTS
- U7 pad 13: UART_CTS -> UART2_CTS
- U7 pad 2: OSC -> /UART/OSC1
- U7 pad 3: OSC -> /UART/OSC2
- U7 pad 5: TxLED -> /UART/TX_LED
- U7 pad 6: RxLED -> /UART/RX_LED
- X1 pad 1: OSC -> /UART/OSC1
- X1 pad 2: OSC -> /UART/OSC2
Routing:
- net OSC: track 36.0 -> 0.00 mm
- net FLASH_NAND_CS: track 33.0 -> 0.00 mm, vias 2 -> 0
- net FLASH_NOR_CS: track 0.00 -> 31.6 mm, vias 0 -> 2
- net FLASH_CS: track 28.3 -> 57.9 mm, vias 3 -> 2
- net Net-(SW1-B): track 26.2 -> 0.00 mm, vias 2 -> 0
- net UART_CTS: track 24.6 -> 0.00 mm
- net UART2_CTS: track 0.00 -> 23.5 mm
- net UART_RTS: track 21.7 -> 0.00 mm
- net BOOT0: track 27.0 -> 47.9 mm
- net UART2_RTS: track 0.00 -> 19.2 mm
- net SPI1_MISO: track 29.2 -> 48.4 mm, vias 3 -> 0
- net Net-(U2-HOLD(IO_{3})): track 0.00 -> 18.5 mm
- net /UART/RX_LED: track 0.00 -> 18.3 mm
- net RxLED: track 18.1 -> 0.00 mm
- net Net-(U3-HOLD(IO_{3})): track 0.00 -> 17.6 mm
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Other:
- board size 75 x 40 mm -> 80 x 50 mm
- board text added: "I2C1"
- board text added: "KabelitzJ STM32G0 Dev Board Rev 1 29.10.2024"

Commit message: asdfsa
Parts:
- added R11: 22, Resistor_SMD:R_0603_1608Metric, F.Cu at (137.9, 111.2)
- added R12: 5k1, Resistor_SMD:R_0603_1608Metric, F.Cu at (132.8, 95.2)
- added R13: 5k1, Resistor_SMD:R_0603_1608Metric, F.Cu at (136.3, 95.3)
- R10: value 10k -> 56k
- moved R10 1.65 mm to (135.4, 110.4), turned to 180 degrees
- moved R7 1.55 mm to (127.9, 92.3)
Connections:
- C1 pad 1: +5V_USB -> Net-(U6-IN)
- U2 pad 8: SPI1_MISO -> /FLASH/SPI1_MISO
- U3 pad 8: SPI1_MISO -> /FLASH/SPI1_MISO
- U6 pad 1: +5V_USB -> Net-(U6-IN)
Routing:
- net +3.3V: track 43.7 -> 46.2 mm, vias 16 -> 18
- net SPI1_SCK: track 39.2 -> 37.8 mm, vias 4 -> 2
- net Net-(U2-HOLD(IO_{3})): track 18.5 -> 17.5 mm
- net I2C1_SDA: track 24.1 -> 23.4 mm

Commit message: asdfsa
Parts:
- removed C1: 1u, Capacitor_SMD:C_0603_1608Metric
- removed C2: 10u, Capacitor_SMD:C_0603_1608Metric
- removed U6: ~, custom:TPS7B8333QDCYRQ1
- removed X1: 12M, custom:73-XT49M1200-S
- added C17: 100n, Capacitor_SMD:C_0603_1608Metric, F.Cu at (118.5, 99.3)
- added C18: 4u7, Capacitor_SMD:C_0603_1608Metric, F.Cu at (122.9, 100.1)
- added FB2: FerriteBead, Capacitor_SMD:C_0603_1608Metric, F.Cu at (114.0, 98.9)
- added R18: 270, Resistor_SMD:R_0603_1608Metric, F.Cu at (116.0, 114.8)
- C11, C3, C4: value C -> 47p
- R4: value 4k7 -> 27
- R5: value R -> 27
- R6: value R -> 270
- U7: value MCP2200-I-SO -> FT230XS; footprint Package_SO:SOIC-20W_7.5x12.8mm_P1.27mm -> Package_SO:SSOP-16_3.9x4.9mm_P0.635mm
- moved C4 22.5 mm to (115.8, 102.3), turned to 90 degrees
- moved C3 21.3 mm to (115.8, 105.4)
- moved R5 16.3 mm to (118.3, 104.7), turned to 0 degrees
- moved R3 15.8 mm to (120.7, 94.1), turned to 180 degrees
- moved D3 14.6 mm to (116.0, 119.7)
- moved C13 13.5 mm to (109.2, 114.6), turned to 90 degrees
- moved D1 11.6 mm to (116.3, 94.1), turned to 180 degrees
- moved H4 11.2 mm to (105.0, 120.0)
- moved SW2 10.8 mm to (105.0, 113.9), turned to 0 degrees
- moved R1 10.3 mm to (111.4, 101.2)
- moved R2 10.3 mm to (111.4, 104.2)
- moved U4 10.3 mm to (103.3, 102.5)
- moved C11 10.2 mm to (125.8, 98.7), turned to 90 degrees
- moved R4 10.0 mm to (118.3, 103.1), turned to 0 degrees
- moved H1 10.0 mm to (105.0, 85.0)
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Connections:
- net UART1_CTS renamed ~{UART1_CTS}
- net UART1_RTS renamed ~{UART1_RTS}
- C11 pad 1: +3.3V -> Net-(U7-~{RESET})
- C3 pad 1: /UART/OSC1 -> USB_D+
- C4 pad 1: /UART/OSC2 -> USB_D-
- R4 pad 1: +3.3V -> USB_D-
- R4 pad 2: /UART/RST -> USB_D-
- R5 pad 1: /UART/TX_LED -> USB_D+
- R5 pad 2: Net-(D2-A) -> USB_D+
- R6 pad 1: /UART/RX_LED -> /POWER_SUPPLY/TX_LED
- R6 pad 2: Net-(D3-A) -> Net-(D2-A)
- U1 pad 7: UART2_CTS -> ~{UART2_CTS}
- U1 pad 8: UART2_RTS -> ~{UART2_RTS}
- U2 pad 8: /FLASH/SPI1_MISO -> SPI1_MISO
- U3 pad 8: /FLASH/SPI1_MISO -> SPI1_MISO
- U7 pad 1: +3.3V -> UART2_TX
- U7 pad 10: UART2_TX -> +3.3V
- U7 pad 11: UART2_RTS -> Net-(U7-~{RESET})
- U7 pad 12: UART2_RX -> +5V_USB
- U7 pad 13: UART2_CTS -> GND
- U7 pad 14: unconnected-(U7-GP2-Pad14) -> /POWER_SUPPLY/RX_LED
- U7 pad 2: /UART/OSC1 -> ~{UART2_RTS}
- U7 pad 3: /UART/OSC2 -> +3.3V
- U7 pad 4: /UART/RST -> UART2_RX
- U7 pad 5: /UART/TX_LED -> GND
- U7 pad 6: /UART/RX_LED -> ~{UART2_CTS}
- U7 pad 7: unconnected-(U7-GP5-Pad7) -> /POWER_SUPPLY/TX_LED
- U7 pad 8: unconnected-(U7-GP4-Pad8) -> USB_D+
- U7 pad 9: unconnected-(U7-GP3-Pad9) -> USB_D-
Routing:
- net UART2_CTS: track 23.5 -> 0.00 mm
- net UART2_RTS: track 19.2 -> 0.00 mm
- net /UART/RX_LED: track 18.3 -> 0.00 mm
- net /UART/OSC2: track 16.9 -> 0.00 mm
- net /UART/OSC1: track 16.9 -> 0.00 mm
- net ~{UART2_RTS}: track 0.00 -> 15.6 mm
- net /UART/TX_LED: track 15.4 -> 0.00 mm
- net /POWER_SUPPLY/TX_LED: track 0.00 -> 14.7 mm, vias 0 -> 2
- net /POWER_SUPPLY/RX_LED: track 0.00 -> 14.2 mm, vias 0 -> 2
- net NRST: track 44.9 -> 31.0 mm
- net ~{UART2_CTS}: track 0.00 -> 12.1 mm
- net UART2_RX: track 26.9 -> 16.2 mm
- net +3.3V: track 46.2 -> 36.6 mm, vias 18 -> 16
- net +5V_USB: track 18.3 -> 25.8 mm
- net USB_D-: track 26.6 -> 21.8 mm
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- added copper zone on F.Cu, net GND
Other:
- board size 80 x 50 mm -> 70 x 45 mm
- board text added: "KabelitzJ STM32G0 Dev Board Rev. 1 29.10.2024"
- board text removed: "KabelitzJ STM32G0 Dev Board Rev 1 29.10.2024"

Commit message: asdfsa
Parts:
- moved SW1 0.98 mm to (105.8, 92.3)
- moved H2 0.05 mm to (165.0, 85.0)
Connections:
- D2 pad 2: Net-(D2-A) -> /POWER_SUPPLY/TX_LED
- D3 pad 2: Net-(D3-A) -> /POWER_SUPPLY/RX_LED
- R18 pad 2: Net-(D3-A) -> /POWER_SUPPLY/RX_LED
- R6 pad 2: Net-(D2-A) -> /POWER_SUPPLY/TX_LED
Routing:
- net /POWER_SUPPLY/TX_LED: track 14.7 -> 17.3 mm
- net Net-(D3-A): track 2.57 -> 0.00 mm
- net Net-(D2-A): track 2.57 -> 0.00 mm
- net /POWER_SUPPLY/RX_LED: track 14.2 -> 16.8 mm
Other:
- board text added: "3V3"
- board text added: "GND"

Commit message: fsdgds
Parts:
- moved R18 5.47 mm to (116.0, 120.3), turned to 90 degrees
- moved R6 5.47 mm to (121.8, 120.3), turned to 90 degrees
- moved D2 4.18 mm to (121.8, 115.5), turned to 90 degrees
- moved D3 4.18 mm to (116.0, 115.5), turned to 90 degrees
Connections:
- D2 pad 1: GND -> /POWER_SUPPLY/TX_LED
- D2 pad 2: /POWER_SUPPLY/TX_LED -> +3.3V
- D3 pad 1: GND -> /POWER_SUPPLY/RX_LED
- D3 pad 2: /POWER_SUPPLY/RX_LED -> +3.3V
- R18 pad 1: /POWER_SUPPLY/RX_LED -> +3.3V
- R18 pad 2: /POWER_SUPPLY/RX_LED -> +3.3V
- R6 pad 1: /POWER_SUPPLY/TX_LED -> +3.3V
- R6 pad 2: /POWER_SUPPLY/TX_LED -> +3.3V
Routing:
- net +3.3V: track 36.2 -> 47.2 mm, vias 16 -> 17
- net GND: track 66.3 -> 60.5 mm, vias 29 -> 28
- net /POWER_SUPPLY/RX_LED: track 16.8 -> 14.2 mm
- net /POWER_SUPPLY/TX_LED: track 17.3 -> 14.7 mm

Commit message: dssfds
Parts:
- moved R12 0.28 mm to (132.8, 95.5)
- moved R13 0.23 mm to (136.3, 95.5)
- moved R9 0.15 mm to (148.7, 92.9)
Changed lines of the file:
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@@
 	(footprint "Resistor_SMD:R_0603_1608Metric"
 		(layer "F.Cu")
-		(at 148.5 92.925)
+		(at 148.65 92.925)
 		(descr "Resistor SMD 0603 (1608 Metric), square (rectangular) end terminal, IPC_7351 nominal, (Body size source: IPC-SM-782 page 72, https://www.pcb-3d.com/wordpress/wp-content/uploads/ipc-sm-782a_amendment_1_and_2.pdf), generated with kicad-footprint-generator")
 		(tags "resistor")
@@
 	(footprint "Resistor_SMD:R_0603_1608Metric"
 		(layer "F.Cu")
-		(at 136.275 95.3)
+		(at 136.275 95.525)
 		(descr "Resistor SMD 0603 (1608 Metric), square (rectangular) end terminal, IPC_7351 nominal, (Body size source: IPC-SM-782 page 72, https://www.pcb-3d.com/wordpress/wp-content/uploads/ipc-sm-782a_amendment_1_and_2.pdf), generated with kicad-footprint-generator")
 		(tags "resistor")
@@
 	(footprint "Resistor_SMD:R_0603_1608Metric"
 		(layer "F.Cu")
-		(at 132.825 95.25 180)
+		(at 132.825 95.525 180)
 		(descr "Resistor SMD 0603 (1608 Metric), square (rectangular) end terminal, IPC_7351 nominal, (Body size source: IPC-SM-782 page 72, https://www.pcb-3d.com/wordpress/wp-content/uploads/ipc-sm-782a_amendment_1_and_2.pdf), generated with kicad-footprint-generator")
 		(tags "resistor")
@@
 	)
 	(segment
-		(start 147.675 92.925)
-		(end 146.6 92.925)
-		(width 0.5)
-		(layer "F.Cu")
-		(net 2)
-	)
-	(segment
 		(start 134.6 110.45)
 		(end 133.35 110.45)
@@
 	)
 	(segment
-		(start 132 95.25)
-		(end 130.7 95.25)
+		(start 132 95.525)
+		(end 130.7 95.525)
 		(width 0.5)
 		(layer "F.Cu")
@@
 	)
 	(segment
-		(start 137.1 95.3)
-		(end 138.35 95.3)
+		(start 137.1 95.525)
+		(end 138.35 95.525)
 		(width 0.5)
 		(layer "F.Cu")
@@
 	)
 	(segment
+		(start 146.8 92.925)
+		(end 147.825 92.925)
+		(width 0.5)
+		(layer "F.Cu")
+		(net 2)
+	)
+	(segment
 		(start 118.775 121.075)
 		(end 118.77 121.07)
@@
 	)
 	(segment
-		(start 146.15 107.6)
-		(end 147.5 107.6)
+		(start 129.195 102.25)
+		(end 129.2 102.255)
 		(width 0.5)
 		(layer "F.Cu")
@@
 	)
 	(segment
-		(start 116 116.9)
-		(end 116 119.475)
+		(start 146.15 107.6)
+		(end 147.5 107.6)
 		(width 0.5)
 		(layer "F.Cu")
@@
 	)
 	(segment
-		(start 129.2 102.255)
-		(end 127.88 102.255)
+		(start 116 116.9)
+		(end 116 119.475)
 		(width 0.5)
 		(layer "F.Cu")
@@
 	)
 	(segment
+		(start 128.1 102.25)
+		(end 129.195 102.25)
+		(width 0.5)
+		(layer "F.Cu")
+		(net 2)
+	)
+	(segment
 		(start 137.84 121.955)
 		(end 136.34 121.955)
@@
 		(net 2)
 	)
-	(segment
-		(start 127.88 102.255)
-		(end 127.875 102.25)
-		(width 0.5)
-		(layer "F.Cu")
-		(net 2)
-	)
 	(via blind
 		(at 122.9775 109.1)
@@
 	)
 	(via blind
-		(at 130.7 95.25)
+		(at 130.7 95.525)
 		(size 0.6)
 		(drill 0.3)
@@
 	)
 	(via blind
-		(at 127.875 102.25)
+		(at 128.1 102.25)
 		(size 0.6)
 		(drill 0.3)
@@
 	)
 	(via blind
-		(at 138.35 95.3)
+		(at 138.35 95.525)
 		(size 0.6)
 		(drill 0.3)
@@
 	)
 	(via blind
-		(at 146.6 92.925)
+		(at 146.8 92.925)
 		(size 0.6)
 		(drill 0.3)
@@
 	)
 	(segment
-		(start 109.835661 98.875)
+		(start 110.575 98.875)
 		(end 113.275 98.875)
 		(width 0.5)
@@
 	)
 	(segment
-		(start 107.3 100.25)
-		(end 108.460661 100.25)
+		(start 117.29 98.875)
+		(end 118.52 100.105)
 		(width 0.5)
 		(layer "F.Cu")
@@
 	)
 	(segment
-		(start 117.29 98.875)
-		(end 118.52 100.105)
+		(start 109.2 100.25)
+		(end 110.575 98.875)
 		(width 0.5)
 		(layer "F.Cu")
@@
 	)
 	(segment
-		(start 124.245 101.885)
-		(end 124.245 102.65)
+		(start 107.3 100.25)
+		(end 109.2 100.25)
 		(width 0.5)
 		(layer "F.Cu")
@@
 	)
 	(segment
-		(start 107.3 105.05)
-		(end 107.3 104.877)
+		(start 124.245 101.885)
+		(end 124.245 102.65)
 		(width 0.5)
 		(layer "F.Cu")
@@
 	)
 	(segment
-		(start 106.627 104.877)
+		(start 107.3 105.05)
 		(end 107.3 104.877)
 		(width 0.5)
@@
 	)
 	(segment
-		(start 108.460661 100.25)
-		(end 109.835661 98.875)
+		(start 106.627 104.877)
+		(end 107.3 104.877)
 		(width 0.5)
 		(layer "F.Cu")
@@
 	)
 	(segment
-		(start 107.3 103.25)
-		(end 109.950376 103.25)
+		(start 119.17 104.6925)
+		(end 121.218234 104.6925)
 		(width 0.3)
 		(layer "F.Cu")
@@
 	)
 	(segment
-		(start 126.15 106.485)
-		(end 126.15 107.85)
+		(start 107.3 103.25)
+		(end 109.950376 103.25)
 		(width 0.3)
 		(layer "F.Cu")
@@
 	)
 	(segment
-		(start 120.733234 104.2075)
-		(end 122.130734 105.605)
+		(start 106.421131 102.25)
+		(end 107.3 102.25)
 		(width 0.3)
 		(layer "F.Cu")
@@
 	)
 	(segment
-		(start 106.421131 102.25)
-		(end 107.3 102.25)
-		(width 0.3)
-		(layer "F.Cu")
-		(net 21)
-	)
-	(segment
-		(start 119.17 104.6925)
-		(end 119.882501 104.6925)
+		(start 106.098 102.573131)
+		(end 106.421131 102.25)
 		(width 0.3)
 		(layer "F.Cu")
@@
 	)
 	(segment
-		(start 119.882501 104.6925)
-		(end 120.367501 104.2075)
+		(start 115.76 104.6025)
+		(end 117.43 104.6025)
 		(width 0.3)
 		(layer "F.Cu")
@@
 	)
 	(segment
-		(start 106.098 102.573131)
-		(end 106.421131 102.25)
+		(start 106.098 102.926869)
+		(end 106.098 102.573131)
 		(width 0.3)
 		(layer "F.Cu")
@@
 	)
 	(segment
-		(start 120.367501 104.2075)
-		(end 120.733234 104.2075)
+		(start 121.218234 104.6925)
+		(end 122.130734 105.605)
 		(width 0.3)
 		(layer "F.Cu")
@@
 	)
 	(segment
-		(start 115.76 104.6025)
-		(end 117.43 104.6025)
-		(width 0.3)
-		(layer "F.Cu")
-		(net 21)
-	)
-	(segment
-		(start 106.098 102.926869)
-		(end 106.098 102.573131)
+		(start 126.15 106.485)
+		(end 126.15 107.85)
 		(width 0.3)
 		(layer "F.Cu")
@@
 	)
 	(segment
-		(start 144.625 101.325)
-		(end 144.625 90.025)
-		(width 0.3)
-		(layer "F.Cu")
-		(net 29)
-	)
-	(segment
 		(start 141.625 102.69)
 		(end 143.26 102.69)
@@
 	)
 	(segment
-		(start 152.54 84.765)
+		(start 152.54 84.535)
 		(end 152.54 83)
 		(width 0.3)
@@
 	)
 	(segment
-		(start 152.55 85.025)
-		(end 152.55 84.775)
+		(start 150.575 86.5)
+		(end 152.54 84.535)
 		(width 0.3)
 		(layer "F.Cu")
@@
 	)
 	(segment
-		(start 148.15 86.5)
-		(end 151.075 86.5)
-		(width 0.3)
-		(layer "F.Cu")
-		(net 29)
-	)
-	(segment
-		(start 152.55 84.775)
-		(end 152.54 84.765)
+		(start 144.625 101.325)
+		(end 144.625 90.025)
 		(width 0.3)
 		(layer "F.Cu")
@@
 	)
 	(segment
-		(start 151.075 86.5)
-		(end 152.55 85.025)
+		(start 148.15 86.5)
+		(end 150.575 86.5)
 		(width 0.3)
 		(layer "F.Cu")
@@
 	)
 	(segment
-		(start 154.525 92.925)
+		(start 149.475 92.925)
 		(end 151.575 92.925)
 		(width 0.5)
@@
 	)
 	(segment
-		(start 160.875 101.815)
-		(end 159.49 101.815)
+		(start 154.525 92.925)
+		(end 151.575 92.925)
 		(width 0.5)
 		(layer "F.Cu")
@@
 	)
 	(segment
-		(start 149.325 92.925)
-		(end 151.575 92.925)
+		(start 160.875 101.815)
+		(end 159.49 101.815)
 		(width 0.5)
 		(layer "F.Cu")
@@
 	)
 	(segment
-		(start 120.981766 103.6075)
-		(end 122.379266 105.005)
-		(width 0.3)
-		(layer "F.Cu")
-		(net 58)
-	)
-	(segment
 		(start 126.15 104.125)
 		(end 126.15 102.65)
@@
 	)
 	(segment
-		(start 122.379266 105.005)
-		(end 125.27 105.005)
-		(width 0.3)
-		(layer "F.Cu")
-		(net 58)
-	)
-	(segment
 		(start 114.456029 102.45)
 		(end 115.093529 103.0875)
@@
 	)
 	(segment
-		(start 120.367501 103.6075)
-		(end 120.981766 103.6075)
+		(start 107.3 102.75)
+		(end 108.102 102.75)
 		(width 0.3)
 		(layer "F.Cu")
@@
 	)
 	(segment
-		(start 107.3 102.75)
-		(end 108.102 102.75)
+		(start 119.17 103.1225)
+		(end 120.496766 103.1225)
 		(width 0.3)
 		(layer "F.Cu")
@@
 	)
 	(segment
-		(start 119.882501 103.1225)
-		(end 120.367501 103.6075)
+		(start 120.496766 103.1225)
+		(end 122.379266 105.005)
 		(width 0.3)
 		(layer "F.Cu")
@@
 	)
 	(segment
-		(start 125.27 105.005)
-		(end 126.15 104.125)
+		(start 110.150376 102.45)
+		(end 114.456029 102.45)
 		(width 0.3)
 		(layer "F.Cu")
@@
 	)
 	(segment
-		(start 110.150376 102.45)
-		(end 114.456029 102.45)
+		(start 109.950376 102.25)
+		(end 110.150376 102.45)
 		(width 0.3)
 		(layer "F.Cu")
@@
 	)
 	(segment
-		(start 119.17 103.1225)
-		(end 119.882501 103.1225)
+		(start 125.27 105.005)
+		(end 126.15 104.125)
 		(width 0.3)
 		(layer "F.Cu")
@@
 	)
 	(segment
-		(start 109.950376 102.25)
-		(end 110.150376 102.45)
+		(start 122.379266 105.005)
+		(end 125.27 105.005)
 		(width 0.3)
 		(layer "F.Cu")
