File: stm32G0_mcu.kicad_pcb (KiCad board)
At the start: 4 copper layers, 70 x 45 mm, 44 parts, among them J1 Conn_01x04_Pin, J2 Conn_01x06_Pin, J3 Conn_01x04_Pin, SW1 SW_Nidec_CAS-120A1, SW2 SW_Push, U1 STM32G0B0KETx, U7 FT230XS

Commit message: asdfsa
Parts:
- U4: footprint custom:UJ20-C-H-C-MSMT-TR -> custom:640-USB4215-03-A
- moved R1 1.10 mm to (110.3, 101.2)
- moved R2 1.10 mm to (110.3, 104.2)
- moved U4 0.65 mm to (102.7, 102.5)
Connections:
- D2 pad 2: /POWER_SUPPLY/TX_LED -> Net-(D2-A)
- D3 pad 2: /POWER_SUPPLY/RX_LED -> Net-(D3-A)
- R18 pad 2: /POWER_SUPPLY/RX_LED -> Net-(D3-A)
- R6 pad 2: /POWER_SUPPLY/TX_LED -> Net-(D2-A)
Routing:
- net Net-(D3-A): track 0.00 -> 2.57 mm
- net Net-(D2-A): track 0.00 -> 2.57 mm
- net /POWER_SUPPLY/RX_LED: track 16.8 -> 14.2 mm
- net /POWER_SUPPLY/TX_LED: track 17.3 -> 14.7 mm
- net /POWER_SUPPLY/CC: track 6.55 -> 5.61 mm
- net +5V_USB: track 25.8 -> 26.5 mm
Other:
- board text added: "CLK"
- board text added: "IO"
- board text added: "SCL"
- board text added: "SDA"
- board text added: "VCC"
